Commit message: grados entre arduino y simulacion

File: src/ros2_ws/src/robot_pkg/urdf/robotfisico.urdf (robot description, URDF)
Before this commit: robot brazo_fisico_pinza_mixta_invertido, 8 links, 7 joints
Joints:
- joint joint_c3_to_izq: limit lower=-0.78 upper=0.78 effort=1.0 velocity=2.0 -> lower=-1.57 upper=1.57 effort=1.0 velocity=2.0
