Commit message: Mejorado TCP, falta comprobar todo el funcinamiento

File: src/ros2_ws/src/robot_pkg/urdf/robot.urdf (robot description, URDF)
Before this commit: robot robot_cilindros_pinza_simple, 8 links, 7 joints
Links:
- removed link dedo_der
- removed link dedo_izq
- added link c4_muneca; visual cylinder length=0.1 radius=0.05
- link c1_base: mass 1.0 -> None
- link c2_brazo: mass 1.0 -> None
- link c3_antebrazo: mass 1.0 -> None
- link c5_muneca2_gira: mass 1.0 -> None; geometry collision cylinder length=0.1 radius=0.05; visual cylinder length=0.1 radius=0.05
- link mano: mass 1.0 -> None; geometry visual box size=0.05 0.01 0.07
Joints:
- removed joint joint_c3_c5
- removed joint joint_dedo_der_fijo
- removed joint joint_pinza
- added joint joint_c3_c4: type revolute, parent c3_antebrazo, child c4_muneca, origin xyz=0 0 0.3 rpy=0 0 0, axis 0 1 0, limit lower=-1.57 upper=1.57 effort=0.25 velocity=2.0
- added joint joint_c4_c5: type revolute, parent c4_muneca, child c5_muneca2_gira, origin xyz=0 0 0.1 rpy=0 0 0, axis 0 0 1, limit lower=-1.57 upper=1.57 effort=0.25 velocity=2.0
- joint joint_base_c1: limit lower=-1.57 upper=1.57 effort=10 velocity=2.0 -> lower=-1.57 upper=1.57 effort=0.25 velocity=2.0; origin xyz=0 0 0.2 -> xyz=0 0 0.2 rpy=0 0 0
- joint joint_c1_c2: limit lower=-1.57 upper=1.57 effort=10 velocity=2.0 -> lower=-1.57 upper=1.57 effort=0.25 velocity=2.0; origin xyz=0 0 0.2 -> xyz=0 0 0.2 rpy=0 0 0
- joint joint_c2_c3: limit lower=-1.57 upper=1.57 effort=10 velocity=2.0 -> lower=-1.57 upper=1.57 effort=0.25 velocity=2.0; origin xyz=0 0 0.3 -> xyz=0 0 0.3 rpy=0 0 0

Commit message: Version mejorada 3 en raya no probada, version anterior si va pero sin moverse ceo

File: src/ros2_ws/src/robot_pkg/urdf/robot.urdf (robot description, URDF)
Before this commit: robot robot_cilindros, 7 links, 6 joints
Links:
- link base: geometry collision cylinder length=0.2 radius=0.1; visual cylinder length=0.2 radius=0.1

Commit message: Añadido cambiar de robot con config, solucionado bug 3 en raya, nuevo robot con nueva tcp default, comprobar de nuevo comandos

File: src/ros2_ws/src/robot_pkg/urdf/robot.urdf (robot description, URDF)
Before this commit: robot robot_cilindros, 7 links, 6 joints
Links:
- added link c6_herramienta; visual cylinder length=0.05 radius=0.05
- link c5_muneca2_gira: geometry visual cylinder length=0.1 radius=0.05
Joints:
- removed joint joint_c5_mano
- added joint joint_c5_c6: type revolute, parent c5_muneca2_gira, child c6_herramienta, origin xyz=0 0 0.1 rpy=0 0 0, axis 0 0 1, limit lower=-3.14 upper=3.14 effort=0.25 velocity=2.0
- added joint joint_c6_mano: type fixed, parent c6_herramienta, child mano, origin xyz=0 0 0.05 rpy=0 0 0
- joint joint_base_c1: limit lower=-1.57 upper=1.57 effort=0.25 velocity=2.0 -> lower=-3.14 upper=3.14 effort=0.25 velocity=2.0
- joint joint_c1_c2: limit lower=-1.57 upper=1.57 effort=0.25 velocity=2.0 -> lower=-3.14 upper=3.14 effort=0.25 velocity=2.0
- joint joint_c2_c3: limit lower=-1.57 upper=1.57 effort=0.25 velocity=2.0 -> lower=-3.14 upper=3.14 effort=0.25 velocity=2.0
- joint joint_c3_c4: axis 0 1 0 -> 0 0 1; limit lower=-1.57 upper=1.57 effort=0.25 velocity=2.0 -> lower=-3.14 upper=3.14 effort=0.25 velocity=2.0
- joint joint_c4_c5: axis 0 0 1 -> 0 1 0; limit lower=-1.57 upper=1.57 effort=0.25 velocity=2.0 -> lower=-3.14 upper=3.14 effort=0.25 velocity=2.0

Commit message: Correcciones de rutinas, van todas

File: src/ros2_ws/src/robot_pkg/urdf/robot.urdf (robot description, URDF)
Before this commit: robot brazo_fisico_pinza_mixta_invertido, 8 links, 7 joints
Links:
- removed link base_link
- removed link cilindro_1
- removed link cilindro_2
- removed link cilindro_3
- removed link eslabon_final_der
- removed link eslabon_final_izq
- removed link herramienta_fija_der
- removed link herramienta_fija_izq
- added link base, mass 1.0; collision cylinder length=0.2 radius=0.1; visual cylinder length=0.2 radius=0.1
- added link c1_base; visual cylinder length=0.2 radius=0.1
- added link c2_brazo; visual cylinder length=0.3 radius=0.05
- added link c3_antebrazo; visual cylinder length=0.3 radius=0.05
- added link c4_muneca; visual cylinder length=0.1 radius=0.05
- added link c5_muneca2_gira; visual cylinder length=0.1 radius=0.05
- added link c6_herramienta; visual cylinder length=0.05 radius=0.05
- added link mano; visual box size=0.05 0.01 0.07
Joints:
- removed joint joint_base_to_c1
- removed joint joint_c1_to_c2
- removed joint joint_c2_to_c3
- removed joint joint_c3_to_der
- removed joint joint_c3_to_izq
- removed joint joint_der_to_herramienta
- removed joint joint_izq_to_herramienta
- added joint joint_base_c1: type revolute, parent base, child c1_base, origin xyz=0 0 0.2 rpy=0 0 0, axis 0 0 1, limit lower=-3.14 upper=3.14 effort=0.25 velocity=2.0
- added joint joint_c1_c2: type revolute, parent c1_base, child c2_brazo, origin xyz=0 0 0.2 rpy=0 0 0, axis 0 1 0, limit lower=-3.14 upper=3.14 effort=0.25 velocity=2.0
- added joint joint_c2_c3: type revolute, parent c2_brazo, child c3_antebrazo, origin xyz=0 0 0.3 rpy=0 0 0, axis 0 1 0, limit lower=-3.14 upper=3.14 effort=0.25 velocity=2.0
- added joint joint_c3_c4: type revolute, parent c3_antebrazo, child c4_muneca, origin xyz=0 0 0.3 rpy=0 0 0, axis 0 0 1, limit lower=-3.14 upper=3.14 effort=0.25 velocity=2.0
- added joint joint_c4_c5: type revolute, parent c4_muneca, child c5_muneca2_gira, origin xyz=0 0 0.1 rpy=0 0 0, axis 0 1 0, limit lower=-3.14 upper=3.14 effort=0.25 velocity=2.0
- added joint joint_c5_c6: type revolute, parent c5_muneca2_gira, child c6_herramienta, origin xyz=0 0 0.1 rpy=0 0 0, axis 0 0 1, limit lower=-3.14 upper=3.14 effort=0.25 velocity=2.0
- added joint joint_c6_mano: type fixed, parent c6_herramienta, child mano, origin xyz=0 0 0.05 rpy=0 0 0

Commit message: Mejora wall y solucionde errores

File: src/ros2_ws/src/robot_pkg/urdf/robot.urdf (robot description, URDF)
Before this commit: robot robot_cilindros_6dof, 8 links, 7 joints
Links:
- removed link base
- removed link c1_base
- removed link c2_brazo
- removed link c3_antebrazo
- removed link c4_muneca
- removed link c5_muneca2_gira
- removed link c6_herramienta
- removed link mano
- added link base_link, mass 1.0; collision box size=0.1 0.1 0.04; visual box size=0.1 0.1 0.04
- added link cilindro_1; visual cylinder length=0.03 radius=0.02
- added link cilindro_2; visual cylinder length=0.07 radius=0.02
- added link cilindro_3; visual cylinder length=0.07 radius=0.02
- added link eslabon_final_der; visual cylinder length=0.05 radius=0.005
- added link eslabon_final_izq; visual cylinder length=0.05 radius=0.005
- added link herramienta_fija_der; visual cylinder length=0.055 radius=0.005
- added link herramienta_fija_izq; visual cylinder length=0.055 radius=0.005
Joints:
- removed joint joint_base_c1
- removed joint joint_c1_c2
- removed joint joint_c2_c3
- removed joint joint_c3_c4
- removed joint joint_c4_c5
- removed joint joint_c5_c6
- removed joint joint_c6_mano
- added joint joint_base_to_c1: type revolute, parent base_link, child cilindro_1, origin xyz=0 0 0.04 rpy=0 0 0, axis 0 0 1, limit lower=-1.57 upper=1.57 effort=1.0 velocity=2.0
- added joint joint_c1_to_c2: type revolute, parent cilindro_1, child cilindro_2, origin xyz=0 0 0.03 rpy=0 0 0, axis -1 0 0, limit lower=-1.57 upper=1.57 effort=1.0 velocity=2.0
- added joint joint_c2_to_c3: type revolute, parent cilindro_2, child cilindro_3, origin xyz=0 0 0.07 rpy=0 0 0, axis 1 0 0, limit lower=-1.57 upper=1.57 effort=1.0 velocity=2.0
- added joint joint_c3_to_der: type fixed, parent cilindro_3, child eslabon_final_der, origin xyz=0 0 0.07 rpy=0 -0.9 0
- added joint joint_c3_to_izq: type revolute, parent cilindro_3, child eslabon_final_izq, origin xyz=0 0 0.07 rpy=0 0.7854 0, axis 0 1 0, limit lower=-1.57 upper=1.57 effort=1.0 velocity=2.0
- added joint joint_der_to_herramienta: type fixed, parent eslabon_final_der, child herramienta_fija_der, origin xyz=0 0 0.05 rpy=0 1.5708 0
- added joint joint_izq_to_herramienta: type fixed, parent eslabon_final_izq, child herramienta_fija_izq, origin xyz=0 0 0.05 rpy=0 -1.5708 0
